Commit message: added hada_robot_sim v1

File: h500_description/h500_sprayer/hada_robot_dae_sim_rev0.urdf.xacro (robot description, xacro)
@@ -5,12 +5,18 @@
 <!-- =================================================================================== -->
 <robot name="h500_sprayer">
+  <material name="blue">
+    <color rgba="0 0 0.8 1"/>
+  </material>
+  <material name="yellow">
+    <color rgba="0.8 0.8 0 1"/>
+  </material>
   <!-- =============== Link & Joint =============== -->
   <!-- Base -->
-  <link name="base_footprint"/>
+<!--  <link name="base_footprint"/>
   <joint name="base_link_joint" type="fixed">
     <origin rpy="0 0 0" xyz="0 0 0.15"/>
     <parent link="base_footprint"/>
     <child link="base_link"/>
-  </joint>
+  </joint> -->
   <link name="base_link">
     <visual>
@@ -30,4 +36,32 @@
     </inertial>
   </link>
+<!--marker base link-->
+  <joint name="marker_base_link_joint" type="fixed">
+    <origin rpy="0 0 0" xyz="0 0 0.15"/>
+    <parent link="base_link"/>
+    <child link="marker_base_link"/>
+  </joint>
+  <link name="marker_base_link">
+    <visual>
+      <origin rpy="0 0 0" xyz="0 0 0"/>
+      <geometry>
+        <box size="1.118 0.699 0.1"/>
+      </geometry>
+      <material name="green"/>
+    </visual>
+    <collision>
+      <origin rpy="0 0 0" xyz="0 0 0"/>
+      <geometry>
+        <box size="1.118 0.699 0.1"/> <!-- <box size="0.5 0.3 0.1"/> -->
+      </geometry>
+    </collision>
+    <inertial>
+      <origin rpy="0 0 0" xyz="0 0 0"/>
+      <mass value="5"/>
+      <inertia ixx="0.0416666666667" ixy="0.0" ixz="0.0" iyy="0.108333333333" iyz="0.0" izz="0.141666666667"/>
+    </inertial>
+  </link>
+<!--end of marker base link-->
+<!--editing front right steer-->
   <joint name="front_right_steering_joint" type="revolute">
     <origin xyz="-0.442 0.361 0.0135"/>
@@ -54,4 +88,64 @@
     </inertial>
   </link>
+<!--end of front right steering section -->
+<!-- front right steering steering marker -->
+  <link name="marker_front_right_steer_link">
+    <visual>
+      <origin rpy="0 0 0" xyz="0 0 0"/>
+      <geometry>
+        <cylinder length="0.02" radius="0.1"/>
+      </geometry>
+      <material name="blue"/>
+    </visual>
+    <collision>
+      <origin rpy="0 0 0" xyz="0 0 0"/>
+      <geometry>
+        <cylinder length="0.02" radius="0.20"/>
+      </geometry>
+    </collision>
+    <inertial>
+      <origin rpy="0 0 0" xyz="0 0 0"/>
+      <mass value="1"/>
+      <inertia ixx="0.000658333333333" ixy="0.0" ixz="0.0" iyy="0.000658333333333" iyz="0.0" izz="0.00125"/>
+    </inertial>
+  </link>
+  <joint name="marker_front_right_steer_joint" type="revolute">
+    <parent link="front_right_steering_link"/>
+    <child link="marker_front_right_steer_link"/>
+    <origin rpy="0 0 0" xyz="0 0 0.43"/>
+    <axis xyz="0 0 1"/>
+    <limit effort="10.0" lower="-0.785398163397" upper="0.785398163397" velocity="5.0"/>
+  </joint>
+<!-- end of front right steering steering marker -->
+<!--front steer middle-->
+  <link name="front_steer_link">
+    <visual>
+      <origin rpy="0 0 0" xyz="0 0 0"/>
+      <geometry>
+        <cylinder length="0.02" radius="0.10"/>
+      </geometry>
+      <material name="yellow"/>
+    </visual>
+    <collision>
+      <origin rpy="0 0 0" xyz="0 0 0"/>
+      <geometry>
+        <cylinder length="0.02" radius="0.05"/>
+      </geometry>
+    </collision>
+    <inertial>
+      <origin rpy="0 0 0" xyz="0 0 0"/>
+      <mass value="1"/>
+      <inertia ixx="0.000658333333333" ixy="0.0" ixz="0.0" iyy="0.000658333333333" iyz="0.0" izz="0.00125"/>
+    </inertial>
+  </link>
+  <joint name="front_steer_joint" type="revolute">
+    <parent link="base_link"/>
+    <child link="front_steer_link"/>
+    <origin rpy="0 0 0" xyz="-0.442 0.0 0.45"/> <!-- xyz="0.2 0 0.12 -->
+    <axis xyz="0 0 1"/>
+    <limit effort="10.0" lower="-3.14159265359" upper="3.14159265359" velocity="5.0"/>
+  </joint>
+<!--end of front steer middle-->
+<!--front left steering section -->
   <joint name="front_left_steering_joint" type="revolute">
     <origin xyz="-0.442 -0.3495 0.0135"/>
@@ -78,4 +172,35 @@
     </inertial>
   </link>
+<!--end of front left steering section -->
+<!-- front left steering steering marker -->
+  <link name="marker_front_left_steer_link">
+    <visual>
+      <origin rpy="0 0 0" xyz="0 0 0"/>
+      <geometry>
+        <cylinder length="0.02" radius="0.1"/>
+      </geometry>
+      <material name="blue"/>
+    </visual>
+    <collision>
+      <origin rpy="0 0 0" xyz="0 0 0"/>
+      <geometry>
+        <cylinder length="0.02" radius="0.1"/>
+      </geometry>
+    </collision>
+    <inertial>
+      <origin rpy="0 0 0" xyz="0 0 0"/>
+      <mass value="1"/>
+      <inertia ixx="0.000658333333333" ixy="0.0" ixz="0.0" iyy="0.000658333333333" iyz="0.0" izz="0.00125"/>
+    </inertial>
+  </link>
+  <joint name="marker_front_left_steer_joint" type="revolute">
+    <parent link="front_left_steering_link"/>
+    <child link="marker_front_left_steer_link"/>
+    <origin rpy="0 0 0" xyz="0 0 0.43"/> <!-- <origin rpy="0 0 0" xyz="0 0 0.43"/>-->
+    <axis xyz="0 0 1"/>
+    <limit effort="10.0" lower="-0.785398163397" upper="0.785398163397" velocity="5.0"/>
+  </joint>
+<!-- end of front left steering steering marker -->
+<!--rear right steering section -->
   <joint name="rear_right_steering_joint" type="revolute">
     <origin xyz="0.676 0.361 0.0135"/>
@@ -102,4 +227,6 @@
     </inertial>
   </link>
+<!--end of rear right steering section -->
+<!--rear left steering section -->
   <joint name="rear_left_steering_joint" type="revolute">
     <origin xyz="0.676 -0.3495 0.0135"/>
@@ -126,4 +253,6 @@
     </inertial>
   </link>
+<!--end of rear left steering section -->
+<!--ffr_wheel_joint-->
   <joint name="ffr_wheel_joint" type="continuous">
     <origin rpy="0 0 3.14159274" xyz="-0.0004 0.07 0.118"/>
@@ -150,4 +279,6 @@
     </inertial>
   </link>
+<!--end of ffr wheel section-->
+<!--ffl_wheel_joint-->
   <joint name="ffl_wheel_joint" type="continuous">
     <origin rpy="0 0 3.14159274" xyz="-0.0004 -0.32 0.118"/>
@@ -174,4 +305,6 @@
     </inertial>
   </link>
+<!--end of ffl wheel section-->
+<!--rfr wheel section-->
   <joint name="rfr_wheel_joint" type="continuous">
     <origin rpy="0 0 3.14159274" xyz="-0.0004 0.07 0.118"/>
@@ -198,4 +331,6 @@
     </inertial>
   </link>
+<!--end of rfr wheel section-->
+<!--rfl wheel section-->
   <joint name="rfl_wheel_joint" type="continuous">
     <origin rpy="0 0 3.14159274" xyz="-0.0004 -0.32 0.118"/>
@@ -222,4 +357,46 @@
     </inertial>
   </link>
+<!--end of rfl wheel section-->
+<!--rear wheel link-->
+  <link name="rear_wheel_link">
+    <visual>
+      <origin rpy="0 0 0" xyz="0 0 0"/>
+      <geometry>
+        <cylinder length="0.04" radius="0.1"/> <!-- <cylinder length="0.04" radius="0.025"/> -->
+      </geometry>
+      <material name="yellow"/>
+    </visual>
+    <collision>
+      <origin rpy="0 0 0" xyz="0 0 0"/>
+      <geometry>
+        <cylinder length="0.04" radius="0.1"/> <cylinder length="0.04" radius="0.025"/>
+      </geometry>
+    </collision>
+    <inertial>
+      <origin rpy="0 0 0" xyz="0 0 0"/>
+      <mass value="0.03125"/>
+      <inertia ixx="9.04947916667e-06" ixy="0.0" ixz="0.0" iyy="9.04947916667e-06" iyz="0.0" izz="9.765625e-06"/>
+    </inertial>
+  </link>
+  <joint name="rear_wheel_joint" type="continuous">
+    <parent link="base_link"/>
+    <child link="rear_wheel_link"/>
+    <origin rpy="-1.57079632679 0 0" xyz="0.676 0 0.1315"/>
+    <axis xyz="0 0 1"/>
+  </joint>
+  <transmission name="rear_wheel_joint_trans">
+    <type>transmission_interface/SimpleTransmission</type>
+    <actuator name="rear_wheel_joint_motor">
+      <mechanicalReduction>1</mechanicalReduction>
+      <hardwareInterface>hardware_interface/VelocityJointInterface</hardwareInterface>
+    </actuator>
+    <joint name="rear_wheel_joint">
+      <hardwareInterface>hardware_interface/VelocityJointInterface</hardwareInterface>
+    </joint>
+  </transmission>
+  <gazebo reference="rear_wheel_link">
+    <material>Gazebo/Yellow</material>
+  </gazebo>
+<!--end of rear wheel link-->
   <transmission name="ffr_wheel_trans">
     <type>transmission_interface/SimpleTransmission</type>
