Commit message: updated hada_explorer_Description

File: h500_description/urdf/base/base_base_footprint.urdf.xacro (robot description, xacro)
@@ -2,10 +2,10 @@
 <robot xmlns:xacro="http://ros.org/wiki/xacro">
   <xacro:include filename="$(find h500_description)/urdf/base/base.gazebo.xacro"/>
-  <!-- <xacro:macro name="base_v0" params="parent *joint_origin">
+  <xacro:macro name="base_v0" params="parent *joint_origin">
 	<joint name="base_link_joint" type="fixed">
 	  <xacro:insert_block name="joint_origin"/>
 	  <parent link="${parent}"/>
 	  <child link="base_link"/>
-	</joint> -->
+	</joint>
 	<link name="base_link">
 	  <visual>
@@ -20,9 +20,9 @@
 	  </collision>
 	  <inertial>
-		<origin xyz="0 0 0.5"/> <!-- origin xyz="0 0 0.017 -->
+		<origin xyz="0 0 0.017"/> <!-- origin xyz="0 0 0.017 -->
 		<mass value="1.2"/>
 		<inertia ixx="0.0001873" ixy="0" ixz="0" iyy="0.000055" iyz="0" izz="0.0002283" />
 	  </inertial>
 	</link>
-  <!-- </xacro:macro> -->
+  </xacro:macro>
 </robot>
